File: pcb/TP_Final.sch (KiCad schematic (older format))
At the start: 24 parts, among them J1 Conn_01x07, J2 Conn_01x02, J3 Conn_01x02, U1 MAX98357AETE+T, U2 MAX98357AETE+T

Commit message: Modelos 3D y PCB
Parts:
- C1, C2, C3, C4, C5, C6, C7, C8: footprint Capacitor_SMD:C_0402_1005Metric -> Capacitor_SMD:C_0805_2012Metric; category (none) -> CAP
- FB1, FB2, FB3, FB4: footprint Ferrite_THT:LairdTech_28C0236-0JW-10 -> Fuse:Fuse_0805_2012Metric; category (none) -> FE; digikey part number (none) -> 710-742792030
- J1: footprint Connector_PinSocket_2.54mm:PinSocket_1x07_P2.54mm_Vertical -> Connector_PinHeader_2.54mm:PinHeader_1x07_P2.54mm_Vertical; category (none) -> CONN
- J2, J3: category (none) -> CONN
- R1: footprint Resistor_SMD:R_0402_1005Metric -> Resistor_SMD:R_0805_2012Metric; category (none) -> RF; digikey description (none) -> Resistores de alta frecuencia RF
Connections:
- net at C8.1, FB4.2: now also J3.1 (Pin_1); no longer J3.2 (Pin_2)
- net at C7.1, FB3.2: now also J3.2 (Pin_2); no longer J3.1 (Pin_1)
- net at C6.1, FB2.2: now also J2.1 (Pin_1); no longer J2.2 (Pin_2)
- net at C5.1, FB1.2: now also J2.2 (Pin_2); no longer J2.1 (Pin_1)
