File: pcb/TP_Final.kicad_pcb (KiCad board)
At the start: 2 copper layers, 24 parts, among them J1 Conn_01x07, J2 Conn_01x02, J3 Conn_01x02, U1 MAX98357AETE+T, U2 MAX98357AETE+T

Commit message: Modelos 3D y PCB
Parts:
- C1, C2, C3, C4, C5, C6, C7, C8: footprint Capacitor_SMD:C_0402_1005Metric -> Capacitor_SMD:C_0805_2012Metric
- FB1, FB2, FB3, FB4: footprint Ferrite_THT:LairdTech_28C0236-0JW-10 -> Fuse:Fuse_0805_2012Metric
- FID1: moved to B.Cu
- J1: footprint Connector_PinSocket_2.54mm:PinSocket_1x07_P2.54mm_Vertical -> Connector_PinHeader_2.54mm:PinHeader_1x07_P2.54mm_Vertical; moved to B.Cu
- R1: footprint Resistor_SMD:R_0402_1005Metric -> Resistor_SMD:R_0805_2012Metric
- moved FID1 48.4 mm to (109.5, 91.8)
- moved U1 46.7 mm to (118.0, 98.8)
- moved U2 42.2 mm to (118.0, 105.7)
- moved C1 35.2 mm to (115.2, 93.8)
- moved J2 34.9 mm to (132.5, 99.2), turned to 90 degrees
- moved FID4 34.6 mm to (134.5, 102.2)
- moved FID3 34.2 mm to (119.5, 108.8)
- moved C3 33.8 mm to (115.0, 110.8)
- moved J1 33.7 mm to (110.2, 109.8)
- moved H1 33.1 mm to (132.5, 92.2)
- moved J3 31.7 mm to (132.5, 107.8), turned to 90 degrees
- moved FID2 31.5 mm to (119.5, 101.8)
- moved H2 28.4 mm to (132.5, 112.2)
- moved FB4 28.1 mm to (123.0, 109.8), turned to 270 degrees
- moved FB2 27.6 mm to (123.0, 99.3), turned to 270 degrees
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Connections:
- J2 pad 1: Net-(C5-Pad1) -> Net-(C6-Pad1)
- J2 pad 2: Net-(C6-Pad1) -> Net-(C5-Pad1)
- J3 pad 1: Net-(C7-Pad1) -> Net-(C8-Pad1)
- J3 pad 2: Net-(C8-Pad1) -> Net-(C7-Pad1)
Routing:
- net VCC: track 0.00 -> 86.0 mm
- net GND: track 0.00 -> 76.6 mm, vias 0 -> 10
- net /LRCLK: track 0.00 -> 26.6 mm, vias 0 -> 1
- net /BCLK: track 0.00 -> 18.7 mm, vias 0 -> 1
- net /DIN: track 0.00 -> 16.7 mm, vias 0 -> 1
- net /GAIN: track 0.00 -> 15.7 mm, vias 0 -> 1
- net Net-(C5-Pad1): track 0.00 -> 11.5 mm
- net Net-(C6-Pad1): track 0.00 -> 10.7 mm
- net Net-(C8-Pad1): track 0.00 -> 10.3 mm
- net Net-(C7-Pad1): track 0.00 -> 10.1 mm
- net /SD_MODE: track 0.00 -> 8.42 mm
- net Net-(FB1-Pad1): track 0.00 -> 7.49 mm
- net Net-(FB4-Pad1): track 0.00 -> 4.86 mm
- net Net-(R1-Pad1): track 0.00 -> 4.57 mm
- net Net-(FB3-Pad1): track 0.00 -> 4.30 mm
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- added copper zone on F.Cu, net (none)
- added copper zone on B.Cu, net GND
Other:
- board outline added: 29 x 27 mm
- board text added: "CESE_DCP-TP_FINAL"
- board text added: "Mínimos (Mayer 10mils): Grillas: 1,00 mm; 0,50 mm; 0,25 mm Vía: 1,60 / 0,80 mm Márgen: 0,50 mm Pista: 0,80 mm; 0,25 mm Terminación: HASL Clearance: 0,20 mm Dueño: Lady Ada"
- board text added: "Réplica de adaptador de amplificador Adafruit I2S Clase D"
- board text added: "STACKUP F.Cu________________________ 1oz //////Espesor 1,60 mm////// B.Cu________________________ 1oz"
- board text added: "V.1 14/10/21"

Commit message: Correciones
Other:
- board text added: "Mínimos (Mayer 10mils): Grillas: 1,00 mm; 0,50 mm; 0,25 mm Vía: 0,80 / 0,40 mm Márgen: 0,50 mm Pista: 0,80 mm; 0,25 mm Terminación: HASL Clearance: 0,20 mm Dueño: Lady Ada"
- board text removed: "Mínimos (Mayer 10mils): Grillas: 1,00 mm; 0,50 mm; 0,25 mm Vía: 1,60 / 0,80 mm Márgen: 0,50 mm Pista: 0,80 mm; 0,25 mm Terminación: HASL Clearance: 0,20 mm Dueño: Lady Ada"
